Commit message: Added controllers and tweaked parameters

File: hydrus/hydrus_description/urdf/base.xacro (robot description, xacro)
@@ -12,5 +12,5 @@
     Vehicle's parameters (remember to enter the model parameters below)
   -->
-  <xacro:property name="mass" value="15.3383002922666"/>
+  <xacro:property name="mass" value="18.062"/>
   <!-- Center of gravity -->
   <xacro:property name="cog" value="0 0 0"/>

File: hydrus/hydrus_description/urdf/gazebo.xacro (robot description, xacro)
@@ -4,5 +4,5 @@
     <xacro:property name="hydrus_cob" value="0 0 0"/>
     <!-- Vehicle's actual volume (Gazebo cannot compute the volume out of the mesh) -->
-    <xacro:property name="hydrus_volume" value="0.07"/>
+    <xacro:property name="hydrus_volume" value="0.009"/>
     <!-- Describing the dimensions of the vehicle's bounding box -->
     <xacro:property name="hydrus_length" value="0.80"/>
