Commit message: Delete unnecessary files and update model parameters

File: hydrus/hydrus_description/urdf/actuators.xacro (robot description, xacro)
@@ -8,27 +8,27 @@
           aware that Gazebo does not use the SNAME convention per default.
     -->
-    <xacro:thruster_macro robot_namespace="${namespace}" thruster_id="0">
-        <origin xyz="-0.243781 -0.170089 -0.054898" rpy="0 0 0" />
+    <xacro:thruster_macro robot_namespace="${namespace}" thruster_id="0" prop_mesh="Thruster_0.STL">
+        <origin xyz="0.40734 -0.19848 -0.034179" rpy="0.5236 -1.5708 0" />
     </xacro:thruster_macro>
-    <xacro:thruster_macro robot_namespace="${namespace}" thruster_id="1">
-        <origin xyz="0.210333 -0.17015 -0.054901" rpy="0 0 0" />
+    <xacro:thruster_macro robot_namespace="${namespace}" thruster_id="1" prop_mesh="Thruster_1.STL">
+        <origin xyz="0.40734 0.19853 -0.034179" rpy="0.5236 1.5708 0" />
     </xacro:thruster_macro>
-    <xacro:thruster_macro robot_namespace="${namespace}" thruster_id="2">
-      <origin xyz="0.211836 0.170263 -0.054903" rpy="0 0 0" />
+    <xacro:thruster_macro robot_namespace="${namespace}" thruster_id="2" prop_mesh="Thruster_2.STL">
+      <origin xyz="-0.43926 -0.19848 -0.034179" rpy="2.618 1.5708 0" />
     </xacro:thruster_macro>
-    <xacro:thruster_macro robot_namespace="${namespace}" thruster_id="3">
-      <origin xyz="-0.242183 0.17005 -0.05497" rpy="0 0 0" />
+    <xacro:thruster_macro robot_namespace="${namespace}" thruster_id="3" prop_mesh="Thruster_3.STL">
+      <origin xyz="-0.43926 0.19853 -0.0341" rpy="2.618 -1.5708 0" />
     </xacro:thruster_macro>
-    <xacro:thruster_macro robot_namespace="${namespace}" thruster_id="4">
-      <origin xyz="-0.437206 -0.198902 -0.033183" rpy="1.5707963267948966 0.5880026035475675 -2.158798930342464" />
+    <xacro:thruster_macro robot_namespace="${namespace}" thruster_id="4" prop_mesh="Thruster_4.STL">
+      <origin xyz="0.21106 0.16968 -0.053127" rpy="0 0 0" />
     </xacro:thruster_macro>
-    <xacro:thruster_macro robot_namespace="${namespace}" thruster_id="5">
-      <origin xyz="0.406277 -0.199528 -0.033572" rpy="1.5707963267948966 -0.5880026035475675 -0.982793723247329" />
+    <xacro:thruster_macro robot_namespace="${namespace}" thruster_id="5" prop_mesh="Thruster_5.STL">
+      <origin xyz="-0.43926 0.19853 -0.0341" rpy="0 0 0" />
     </xacro:thruster_macro>
-    <xacro:thruster_macro robot_namespace="${namespace}" thruster_id="6">
-      <origin xyz="0.406277 0.199528 -0.033572" rpy="-1.5707963267948966 -2.7828219865243244 4.35361831027057225" />
+    <xacro:thruster_macro robot_namespace="${namespace}" thruster_id="6" prop_mesh="Thruster_6.STL">
+      <origin xyz="-0.24297 -0.16962 -0.053127" rpy="0 0 3.1416" />
     </xacro:thruster_macro>
-    <xacro:thruster_macro robot_namespace="${namespace}" thruster_id="7">
-      <origin xyz="-0.437082 0.198902 -0.033183" rpy="-1.5707963267948966 -2.7828219865243244 -4.35361831027057225" />
+    <xacro:thruster_macro robot_namespace="${namespace}" thruster_id="7" prop_mesh="Thruster_7.STL">
+      <origin xyz="0.21106 -0.16962 -0.053127" rpy="0 0 3.1416" />
     </xacro:thruster_macro>
 </robot>

File: hydrus/hydrus_description/urdf/base.xacro (robot description, xacro)
@@ -12,5 +12,5 @@
     Vehicle's parameters (remember to enter the model parameters below)
   -->
-  <xacro:property name="mass" value="18.062"/>
+  <xacro:property name="mass" value="17.0395783829616"/>
   <!-- Center of gravity -->
   <xacro:property name="cog" value="0 0 0"/>
@@ -23,5 +23,5 @@
     Open the meshes for the RexROV vehicle in Blender to see an example on the mesh placement.
   -->
-  <xacro:property name="visual_mesh_file" value="file://$(find hydrus_description)/meshes/hydrus.dae"/>
+  <xacro:property name="visual_mesh_file" value="file://$(find hydrus_description)/meshes/base_link.STL"/>
   <!-- Collision geometry mesh, usually in STL format (it is recommended to keep
   this geometry as simple as possible to improve the performance the physics engine
@@ -38,15 +38,15 @@
         <inertial>
           <origin
-            xyz="-0.0112530988980815 0.0132378868039223 -2.68860266712125E-07"
+            xyz="-0.0117233052541944 7.1124481605241E-06 0.00733571544142573"
             rpy="0 0 0" />
-          <mass
-            value="15.3383002922666" />
-          <inertia
-            ixx="0.0706822953893134"
-            ixy="-2.96658977041411E-09"
-            ixz="4.67785743955219E-06"
-            iyy="0.121380901460858"
-            iyz="1.1891293253612E-09"
-            izz="0.134256272071966" />
+            <mass
+              value="17.0395783829616" />
+            <inertia
+              ixx="0.0720341913567931"
+              ixy="-4.66388174692384E-06"
+              ixz="-2.98192347513836E-09"
+              iyy="0.135463514450081"
+              iyz="5.80636474001404E-10"
+              izz="0.122654380562112" />
         </inertial>
         <visual>

File: hydrus/hydrus_description/urdf/gazebo.xacro (robot description, xacro)
@@ -4,9 +4,9 @@
     <xacro:property name="hydrus_cob" value="0 0 0"/>
     <!-- Vehicle's actual volume (Gazebo cannot compute the volume out of the mesh) -->
-    <xacro:property name="hydrus_volume" value="0.009"/>
+    <xacro:property name="hydrus_volume" value="0.176681341"/>
     <!-- Describing the dimensions of the vehicle's bounding box -->
-    <xacro:property name="hydrus_length" value="0.80"/>
-    <xacro:property name="hydrus_width"  value="0.25"/>
-    <xacro:property name="hydrus_height" value="0.35"/>
+    <xacro:property name="hydrus_length" value="0.930"/>
+    <xacro:property name="hydrus_width"  value="0.436"/>
+    <xacro:property name="hydrus_height" value="0.434"/>
     <xacro:macro name="hydrus_hydro_model" params="namespace">
       <!-- List of hydrodynamic models this robot's links -->

File: hydrus/hydrus_description/urdf/snippets.xacro (robot description, xacro)
@@ -15,9 +15,9 @@
   <!-- Thruster joint and link snippet -->
   <xacro:macro name="thruster_macro"
-    params="robot_namespace thruster_id *origin">
+    params="robot_namespace thruster_id prop_mesh *origin">
     <xacro:thruster_module_first_order_basic_fcn_macro
       namespace="${namespace}"
       thruster_id="${thruster_id}"
-      mesh_filename="file://$(find hydrus_description)/meshes/prop.dae"
+      mesh_filename="file://$(find hydrus_description)/meshes/${prop_mesh}"
       dyn_time_constant="0.05"
       rotor_constant="0.026546960744430276">
